File: hardware/pcb/rav4-tcu.kicad_pcb (KiCad board)
At the start: 2 copper layers, 200 x 170 mm, 140 parts, among them J1 PWR, J2 SOL, J3 SIG, J4 LOAD, K1 G2RL-2 12V, K2 G2RL-2 12V, K3 G2RL-2 12V, Q1 IRF4905, Q2 IRF4905, Q3 IRF4905, U1 ULN2803A, U2 LM393, U3 R-78HB5.0, X4 DASH, X5 SCREEN, X6 ATF, X7 SHIFT

Commit message: Build book accuracy pass: fixes from a full read-through
Checked every claim against the board's nets, the firmware's pins and
messages, the calibration helper, the wiring guide and the shopping list.

Errors fixed:
- Mega power header: the board had 7 holes, the book says an 8-pin strip.
  The unused first pin (NC) now has a hole, so a standard strip fits
- Part 11's final check (the full self-test through the plugs) couldn't
  pass: now a power-up check through X1; the full self-test is in 12.4/13.3
- Part 9: how to drill the heatsink, with M3 x 16 screws and nuts
- Shopping list: foam tape for the screen, 11 lever connectors, 3 fuse
  holders, 23 x 10k, a 3.2 mm drill bit, the heatsink screws
- calibrate.py: two messages still used the old perfboard terminal names
- Bags were numbered by the wrong variable

Clarified: 12.4's expected BAD lines; RESTARTS in the BAD table; the screen
core to terminal mapping; red/black probe for no-shorts checks; 5 V range
4.8-5.2 V; the hot test resistor; no tape needed on the Mega's USB socket;
skills for soldered wires and screw terminals; Bag 1-6 to match Step 1-6.

Co-Authored-By: Claude Opus 5.5 <noreply@anthropic.com>
Claude-Session: https://claude.ai/code/session_01ETJrLv4Z1USdoRELecEc2N
Routing:
- net D9: track 338.6 -> 341.2 mm
- net D3: track 250.8 -> 253.4 mm
- net D20: track 252.0 -> 254.5 mm
- net D21: track 311.0 -> 312.3 mm

Commit message: Optimise: 22 fewer board parts, one electronics order (~$50 cheaper)
Board (rev 3, 113 parts instead of 135):
- The 4 pull-downs on the ULN2803A's inputs are gone: each input already
  has 2.7k + 7.2k to ground inside the chip, so a high-Z Mega pin still
  means every driver and relay off. The cross-check now verifies those
  nets go only to ULN2803A inputs.
- The 18 BAT85 clamp diodes are gone. The switch inputs' series resistor
  goes from 1k to 10k: with 100 nF it is a 1 ms filter, and a core
  shorted to 12 V puts at most 0.65 mA into the Mega's own clamps
  (Microchip AN2519 allows 1 mA). The throttle taps already had 10k.
- Placement spread out where the parts went; routed, DRC 0 errors and 0
  unconnected, every real part fits, box fit check passes. Build book: 56
  small steps (was 60); stale step pictures are now cleaned up.
- Firmware waits 20 ms (not 10) for the slower input filters at boot.

Shopping list ($676 -> $624):
- Optos, comparator, sockets, 1N4148s, zeners, resistors (exact values
  and counts), 100 nF and the 1 uF all move into the DigiKey/Mouser
  order as single pieces, instead of packs and kits.
- The separate silicone wire goes: the 18 AWG harness wire is now
  TXL/GXL (125 C), which also suits the dummy-load cable and the runs
  near the transmission.
- Cross-check: every resistor value and count on the list matches the
  board.

Co-Authored-By: Claude Opus 5.5 <noreply@anthropic.com>
Claude-Session: https://claude.ai/code/session_01ETJrLv4Z1USdoRELecEc2N
Parts:
- removed DH1, DH2, DH3, DH4, DH5, DH6, DH7, DL1, DL2, DL3, DL4, DL5, DL6, DL7, DT1, DT2, DT3, DT4: BAT85, D_DO-35_SOD27_P7.62mm_Horizontal
- removed RD1, RD2, RD3, RD4: 10k, R_Axial_DIN0207_L6.3mm_D2.5mm_P10.16mm_Horizontal
- RS1, RS2, RS3, RS4, RS5, RS6, RS7: value 1k -> 10k
- moved CF1 21.6 mm to (58.9, 165.4)
- moved CF2 21.6 mm to (64.0, 165.4)
- moved CF3 21.6 mm to (69.0, 165.4)
- moved CF4 21.6 mm to (74.1, 165.4)
- moved CF5 21.6 mm to (79.2, 165.4)
- moved CF6 21.6 mm to (84.3, 165.4)
- moved CF7 21.6 mm to (89.4, 165.4)
- moved C3 15.2 mm to (124.9, 132.4)
- moved C4 12.7 mm to (132.6, 132.4)
- moved RT2 2.54 mm to (117.3, 132.4)
Routing:
- net GND: track 1119.4 -> 1274.3 mm, vias 0 -> 13
- net D9: track 341.2 -> 238.9 mm, vias 4 -> 3
- net ECU_2: track 272.0 -> 179.2 mm, vias 2 -> 3
- net D6: track 230.5 -> 161.3 mm, vias 4 -> 1
- net ECU_3: track 269.4 -> 209.7 mm, vias 3 -> 2
- net D21: track 312.3 -> 272.9 mm, vias 4 -> 2
- net ECU_1: track 184.3 -> 151.3 mm, vias 3 -> 1
- net +12_LOG: track 109.7 -> 79.2 mm
- net D28: track 208.9 -> 178.4 mm, vias 6 -> 3
- net D8: track 207.8 -> 178.0 mm, vias 0 -> 2
- net D3: track 253.4 -> 280.0 mm, vias 5 -> 3
- net D23: track 239.4 -> 216.5 mm
- net A0: track 71.8 -> 51.4 mm
- net D24: track 216.5 -> 196.2 mm, vias 3 -> 2
- net +12_COIL: track 363.9 -> 383.0 mm, vias 11 -> 1
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Other:
- board text added: "RAV4 TCU rev 3"
- board text removed: "RAV4 TCU rev 2"
